File: sch/heating_controller/main.sch (EAGLE design)
At the start: 59 parts, among them IC1 LM2575, Q1 BS170, Q2 BC548, Q3 BD140, Q4 IRF4905, Q5 BSS84, T1 BC847, T2 BD139, T3 BD139, T4 BD139

Commit message: 
Parts:
- removed C19: 100n, rcl:C-EU025-024X044
- removed C5: 10n, rcl:C-EU025-024X044
- removed JP5: (no value), pinhead:PINHD-1X2
- removed LED1: (no value), led:LED
- removed Q3: BD140, transistor-pnp:BD140
- removed Q4: IRF4905, transistor-power:IRF4905
- removed R10: 10k, rcl:R-EU_0204/2V
- removed R11, R21: 1k, rcl:R-EU_0204/2V
- removed R12: 10, rcl:R-EU_0204/2V
- removed R14, R19: 4k7, rcl:R-EU_0204/2V
- removed R6, R7: (no value), rcl:R-EU_0204/2V
- removed R8: 47kR, rcl:R-EU_0204/2V
- removed R9: 600, rcl:R-EU_0204/2V
- removed T2, T3, T4: BD139, transistor:BD139
- added C10: 100nF, rcl:C-EU025-024X044
- added IC2: 74HC244N, 74xx-eu:74HC244N
- added JP10: (no value), pinhead:PINHD-1X2
- added JP6: (no value), pinhead:PINHD-1X12
- added Q6, Q7, Q8, Q9: IRL2203, transistor-power:IRFZ48Z
- added RN1: 100k, resistor-sil:G04R
- added RN2: 100k, resistor-sil:G08R
- added RN3, RN4: 4k7, resistor-sil:G08R
- added RN6: 100k, resistor-sil:G13R
- JP2: device pinhead:PINHD-1X2 -> pinhead:PINHD-2X24
- JP3: device pinhead:PINHD-1X2 -> pinhead:PINHD-1X12
- JP4: device pinhead:PINHD-1X2 -> pinhead:PINHD-1X16
- L1: value 100uH -> 330uH
- R13: value 1k -> 200R
Connections:
- removed net 1WIRE_TEMP1: JP1.6
- removed net 1WIRE_TEMP2: JP1.8
- removed net CAR_INPUT1_12V: R7.2
- removed net CPU_1WIRE1_INOUT: D2.A, D3.C, R14.1, R15.1
- removed net CPU_1WIRE_SPU: R18.1
- removed net CPU_DIN1: C19.1, JP1.5, R7.1, R8.2
- removed net CPU_DIN2: JP1.7
- removed net CPU_INJECTION: JP1.4
- removed net CPU_STACYJKA: JP1.3
- removed net CPU_VSS: JP1.9
- removed net N$10: JP3.1, Q4.D
- removed net N$11: LED1.A, R21.1
- removed net N$13: JP3.2
- removed net N$14: LED1.C, T4.C
- removed net USER_KEYA: JP1.23
- removed net USER_KEYB: JP1.27
- new net CPU_1WIRE1_DATA: D2.A, D3.C, JP2.7, R15.1, RN3.2
- new net CPU_1WIRE1_SPU: JP2.8, R18.1, RN2.2
- new net CPU_1WIRE2_DATA: JP2.9
- new net CPU_1WIRE2_SPU: JP2.10
- new net CPU_1WIRE3_DATA: JP2.11
- new net CPU_1WIRE3_SPU: JP2.12
- new net CPU_1WIRE4_DATA: JP2.13
- new net CPU_1WIRE4_SPU: JP2.14
- new net CPU_1WIRE5_DATA: JP2.3
- new net CPU_1WIRE5_SPU: JP2.4
- new net CPU_1WIRE6_DATA: JP2.5
- new net CPU_1WIRE6_SPU: JP2.6
- new net CPU_INPUT2: JP2.24
- new net CPU_INPUT3: JP2.25
- new net CPU_INPUT4: JP2.32
- new net CPU_INPUT5: JP2.33
- new net CPU_INPUT6: JP2.36
- new net CPU_INPUT7: JP2.37
- new net CPU_INPUT8: JP2.38
- new net CPU_OUTPUT1: JP2.26
- new net CPU_OUTPUT2: JP2.40
- new net CPU_OUTPUT3: JP2.41
- new net CPU_VALVE2_OUT: IC2A.A2, JP2.44, RN1.3
- new net CPU_VALVE3_OUT: IC2A.A3, JP2.45, RN1.4
- new net CPU_VALVE4_OUT: IC2A.A4, JP2.46, RN1.5
- new net CPU_VALVE5_OUT: JP2.15
- new net CPU_VALVE6_OUT: JP2.16
- new net N$19: IC2A.Y3, Q8.G
- new net N$21: IC2A.Y1, Q6.G
- new net N$23: IC2A.Y4, Q9.G
- new net N$5: IC2A.Y2, Q7.G
- net +24V: now also JP3.1, JP3.3, JP3.5, JP3.7; no longer Q4.S, R11.2, T3.C
- net +3V3: now also JP2.48
- net +5V: now also C10.2, IC2P.VCC, JP2.2, RN2.1, RN3.1, RN4.1; no longer R14.2, R19.1, R21.2, R6.2
- net ?: now also JP6.1; no longer JP4.1
- net CPU_INPUT1: now also JP2.19, RN4.2; no longer R19.2
- net CPU_VALVE1_OUT: now also IC2A.A1, JP2.43, RN1.2; no longer C5.1, R9.1
- net GND: now also C10.1, IC2A.G, IC2P.GND, JP10.2, JP2.1, JP2.47, JP6.2, Q6.S, Q7.S, Q8.S, Q9.S, RN1.1; no longer C19.2, JP2.2, JP5.2, Q3.C, R10.2, R8.1, T2.E, T4.E
- net LCD_A0: now also JP1.4; no longer JP1.14
- net LCD_BLIGHT: now also JP1.8; no longer JP1.28
- net LCD_CNTR: now also JP1.7; no longer JP1.29
- net LCD_E1: now also JP1.3; no longer JP1.15
- net LCD_E2: now also JP1.6; no longer JP1.16
- net LCD_R/W: now also JP1.5; no longer JP1.17
- net LCD_RST: no longer R6.1
- net N$4: now also JP3.8, Q9.D; no longer C5.2, R10.1, R9.2, T2.B, T4.B
- net N$6: now also JP3.6, Q8.D; no longer Q3.B, R11.1, T2.C, T3.B
- net N$7: now also JP3.4, Q7.D; no longer Q4.G, R12.2
- net N$8: now also JP3.2, Q6.D; no longer Q3.E, R12.1, T3.E
- net N$9: now also JP4.1; no longer JP5.1
- net POW+24V: now also JP10.1; no longer JP2.1
Other:
- moved on the sheet: C6, D2, D3, Q5, R15, R18
